File: tapescanner/tapescanner.sch (KiCad schematic (older format))
At the start: 42 parts, among them J0 Barrel_Jack, Q0 TEPT5600, Q1 TEPT5600, Q2 TEPT5600, Q3 TEPT5600, Q4 TEPT5600, Q5 TEPT5600, Q6 TEPT5600, Q7 TEPT5600, Q8 TEPT5600, Q9 TEPT5600

Commit message: Reduce the number of LEDs
Parts:
- removed D5, D6, D7, D8, D9: LED, symbol Device:LED
- removed R5, R6, R7, R8, R9: 150R, symbol Device:R
- renumbered R14 to R10, R15 to R11, R16 to R12, R17 to R13, R18 to R14, R19 to R15, R20 to R5, R10 to R6, R11 to R7, R12 to R8, R13 to R9
Connections:
- wire segments 124 -> 104
Other:
- moved on the sheet: D0, D1, D2, D3, D4, R0, R1, R2, R3, R4

Commit message: Add the microcontroller
Parts:
- added J1: DB9_Female, symbol Connector:DB9_Female
- added J2: AVR-ISP-10, symbol Connector:AVR-ISP-10
- added R16: 10K, symbol Device:R
- added U0: ATmega328P-PU, Package_DIP:DIP-28_W7.62mm, symbol MCU_Microchip_ATmega:ATmega328P-PU
Connections:
- net labels added: PHOTO_0, PHOTO_1, PHOTO_2, PHOTO_3, PHOTO_4, PHOTO_5, PHOTO_6, PHOTO_7, PHOTO_CTRL, PHOTO_SYNC, SERIAL_RX, SERIAL_TX
- wire segments 104 -> 115
- no-connect marks 0 -> 14
Changed lines of the file:
@@
 $EndComp
-Wire Wire Line
-	1950 4750 1950 5550
-Wire Wire Line
-	2450 4750 2450 5550
-Wire Wire Line
-	2950 4750 2950 5550
-Wire Wire Line
-	3450 4750 3450 5550
-Wire Wire Line
-	4450 4750 4450 5550
-Wire Wire Line
-	4950 4750 4950 5550
-Wire Wire Line
-	5450 4750 5450 5550
-Wire Wire Line
-	5950 4750 5950 5550
-Wire Wire Line
-	6450 4750 6450 5550
 Wire Wire Line
 	6200 4950 6200 5050
@@
 $EndComp
 Wire Wire Line
-	3950 4750 3950 5550
-Wire Wire Line
 	3700 5550 3950 5550
 $Comp
@@
 Wire Wire Line
 	1450 6650 1950 6650
+Wire Wire Line
+	6450 4750 6450 5550
+Wire Wire Line
+	5950 4750 5950 5550
+Wire Wire Line
+	5450 4750 5450 5550
+Wire Wire Line
+	4950 4750 4950 5550
+Wire Wire Line
+	4450 4750 4450 5550
+Wire Wire Line
+	3950 4750 3950 5550
+Wire Wire Line
+	3450 4750 3450 5550
+Wire Wire Line
+	2950 4750 2950 5550
+Wire Wire Line
+	2450 4750 2450 5550
+Wire Wire Line
+	1950 4750 1950 5550
+Text Label 1950 4750 1    50   ~ 0
+PHOTO_0
+Text Label 2450 4750 1    50   ~ 0
+PHOTO_1
+Text Label 2950 4750 1    50   ~ 0
+PHOTO_2
+Text Label 3450 4750 1    50   ~ 0
+PHOTO_3
+Text Label 3950 4750 1    50   ~ 0
+PHOTO_4
+Text Label 4450 4750 1    50   ~ 0
+PHOTO_5
+Text Label 4950 4750 1    50   ~ 0
+PHOTO_6
+Text Label 5450 4750 1    50   ~ 0
+PHOTO_7
+Text Label 5950 4750 1    50   ~ 0
+PHOTO_CTRL
+Text Label 6450 4750 1    50   ~ 0
+PHOTO_SYNC
+Text Label 9100 3650 2    50   ~ 0
+PHOTO_0
+Text Label 9100 1250 2    50   ~ 0
+PHOTO_1
+Text Label 9100 1350 2    50   ~ 0
+PHOTO_2
+Text Label 9100 1450 2    50   ~ 0
+PHOTO_3
+Text Label 9100 2950 2    50   ~ 0
+PHOTO_4
+Text Label 9100 2750 2    50   ~ 0
+PHOTO_5
+Text Label 9100 2650 2    50   ~ 0
+PHOTO_6
+Text Label 9100 2550 2    50   ~ 0
+PHOTO_7
+Text Label 9100 2350 2    50   ~ 0
+PHOTO_CTRL
+Text Label 9100 2250 2    50   ~ 0
+PHOTO_SYNC
+$Comp
+L power:GND #PWR0107
+U 1 1 607C97D1
+P 9700 950
+F 0 "#PWR0107" H 9700 700 50  0001 C CNN
+F 1 "GND" H 9705 777 50  0000 C CNN
+F 2 "" H 9700 950 50  0001 C CNN
+F 3 "" H 9700 950 50  0001 C CNN
+	1    9700 950
+	-1   0    0    1
+$EndComp
+$Comp
+L power:+5V #PWR0108
+U 1 1 607CA28C
+P 10300 3650
+F 0 "#PWR0108" H 10300 3500 50  0001 C CNN
+F 1 "+5V" V 10315 3778 50  0000 L CNN
+F 2 "" H 10300 3650 50  0001 C CNN
+F 3 "" H 10300 3650 50  0001 C CNN
+	1    10300 3650
+	0    1    1    0
+$EndComp
+$Comp
+L power:+5V #PWR0109
+U 1 1 607CAF72
+P 9700 3950
+F 0 "#PWR0109" H 9700 3800 50  0001 C CNN
+F 1 "+5V" H 9715 4123 50  0000 C CNN
+F 2 "" H 9700 3950 50  0001 C CNN
+F 3 "" H 9700 3950 50  0001 C CNN
+	1    9700 3950
+	-1   0    0    1
+$EndComp
+$Comp
+L power:+5V #PWR0110
+U 1 1 607CBA93
+P 9600 3950
+F 0 "#PWR0110" H 9600 3800 50  0001 C CNN
+F 1 "+5V" H 9615 4123 50  0000 C CNN
+F 2 "" H 9600 3950 50  0001 C CNN
+F 3 "" H 9600 3950 50  0001 C CNN
+	1    9600 3950
+	-1   0    0    1
+$EndComp
+Wire Wire Line
+	8300 2150 8500 2150
+$Comp
+L Device:R R16
+U 1 1 607D04E2
+P 8150 2150
+F 0 "R16" V 7943 2150 50  0000 C CNN
+F 1 "10K" V 8034 2150 50  0000 C CNN
+F 2 "" V 8080 2150 50  0001 C CNN
+F 3 "~" H 8150 2150 50  0001 C CNN
+	1    8150 2150
+	0    1    1    0
+$EndComp
+$Comp
+L power:+5V #PWR0111
+U 1 1 607D22DC
+P 8000 2150
+F 0 "#PWR0111" H 8000 2000 50  0001 C CNN
+F 1 "+5V" V 8015 2278 50  0000 L CNN
+F 2 "" H 8000 2150 50  0001 C CNN
+F 3 "" H 8000 2150 50  0001 C CNN
+	1    8000 2150
+	0    -1   -1   0
+$EndComp
+$Comp
+L Connector:DB9_Female J1
+U 1 1 607D3CB4
+P 9750 5850
+F 0 "J1" V 9622 6405 50  0000 L CNN
+F 1 "DB9_Female" V 9713 6405 50  0000 L CNN
+F 2 "" H 9750 5850 50  0001 C CNN
+F 3 " ~" H 9750 5850 50  0001 C CNN
+	1    9750 5850
+	0    1    1    0
+$EndComp
+Text Label 9750 5550 1    50   ~ 0
+SERIAL_RX
+Text Label 9950 5550 1    50   ~ 0
+SERIAL_TX
+$Comp
+L power:GND #PWR0112
+U 1 1 607E8C7F
+P 9350 5550
+F 0 "#PWR0112" H 9350 5300 50  0001 C CNN
+F 1 "GND" H 9355 5377 50  0000 C CNN
+F 2 "" H 9350 5550 50  0001 C CNN
+F 3 "" H 9350 5550 50  0001 C CNN
+	1    9350 5550
+	-1   0    0    1
+$EndComp
+Text Label 9100 1850 2    50   ~ 0
+SERIAL_TX
+Text Label 9100 1950 2    50   ~ 0
+SERIAL_RX
+NoConn ~ 9100 1550
+NoConn ~ 9100 1650
+NoConn ~ 9100 1750
+NoConn ~ 9100 2450
+NoConn ~ 9100 3050
+NoConn ~ 9100 3450
+NoConn ~ 9100 3550
+NoConn ~ 9450 5550
+NoConn ~ 9550 5550
+NoConn ~ 9650 5550
+NoConn ~ 9850 5550
+NoConn ~ 10050 5550
+NoConn ~ 10150 5550
+$Comp
+L Connector:AVR-ISP-10 J2
+U 1 1 6081F6F5
+P 8000 3350
+F 0 "J2" H 7670 3446 50  0000 R CNN
+F 1 "AVR-ISP-10" H 7670 3355 50  0000 R CNN
+F 2 "" V 7750 3400 50  0001 C CNN
+F 3 " ~" H 6725 2800 50  0001 C CNN
+	1    8000 3350
+	1    0    0    -1
+$EndComp
+NoConn ~ 7900 2850
+$Comp
+L power:GND #PWR?
+U 1 1 608278F7
+P 7900 3750
+F 0 "#PWR?" H 7900 3500 50  0001 C CNN
+F 1 "GND" H 7905 3577 50  0000 C CNN
+F 2 "" H 7900 3750 50  0001 C CNN
+F 3 "" H 7900 3750 50  0001 C CNN
+	1    7900 3750
+	1    0    0    -1
+$EndComp
+$Comp
+L MCU_Microchip_ATmega:ATmega328P-PU U0
+U 1 1 607AED4A
+P 9700 2450
+F 0 "U0" H 9056 2404 50  0000 R CNN
+F 1 "ATmega328P-PU" H 9056 2495 50  0000 R CNN
+F 2 "Package_DIP:DIP-28_W7.62mm" H 9700 2450 50  0001 C CIN
+F 3 "http://ww1.microchip.com/downloads/en/DeviceDoc/ATmega328_P%20AVR%20MCU%20with%20picoPower%20Technology%20Data%20Sheet%2040001984A.pdf" H 9700 2450 50  0001 C CNN
+	1    9700 2450
+	-1   0    0    1
+$EndComp
+Wire Wire Line
+	8500 3450 8400 3450
+Wire Wire Line
+	8500 3450 8500 2150
+Connection ~ 8500 2150
+Wire Wire Line
+	8500 2150 9100 2150
+Wire Wire Line
+	9100 3150 8900 3350
+Wire Wire Line
+	8900 3350 8400 3350
+Wire Wire Line
+	8400 3250 8900 3250
+Wire Wire Line
+	8900 3250 9000 3350
+Wire Wire Line
+	9000 3350 9100 3350
+Wire Wire Line
+	9100 3250 9000 3150
+Wire Wire Line
+	9000 3150 8400 3150
 $EndSCHEMATC

Commit message: Fine-tune resistors
Parts:
- R10, R11, R12: value 33K -> 120K
- R13, R14, R8: value 33K -> 100K
- R15, R6: value 33K -> 68K
- R7: value 33K -> 47K
- R9: value 33K -> 180K
Other:
- note added: "Fine-tuned"
Changed lines of the file:
@@
 Wire Wire Line
 	6200 5550 6200 5700
-$Comp
-L Device:R R6
-U 1 1 60583FB3
-P 1700 5200
-F 0 "R6" H 1770 5246 50  0000 L CNN
-F 1 "33K" H 1770 5155 50  0000 L CNN
-F 2 "" V 1630 5200 50  0001 C CNN
-F 3 "~" H 1700 5200 50  0001 C CNN
-	1    1700 5200
-	1    0    0    -1
-$EndComp
-$Comp
-L Device:R R7
-U 1 1 6058A786
-P 2200 5200
-F 0 "R7" H 2270 5246 50  0000 L CNN
-F 1 "33K" H 2270 5155 50  0000 L CNN
-F 2 "" V 2130 5200 50  0001 C CNN
-F 3 "~" H 2200 5200 50  0001 C CNN
-	1    2200 5200
-	1    0    0    -1
-$EndComp
 Wire Wire Line
 	6200 4950 6200 5050
@@
 	0    -1   -1   0
 $EndComp
-$Comp
-L Device:R R8
-U 1 1 6058CD3A
-P 2700 5200
-F 0 "R8" H 2770 5246 50  0000 L CNN
-F 1 "33K" H 2770 5155 50  0000 L CNN
-F 2 "" V 2630 5200 50  0001 C CNN
-F 3 "~" H 2700 5200 50  0001 C CNN
-	1    2700 5200
-	1    0    0    -1
-$EndComp
-$Comp
-L Device:R R9
-U 1 1 6058F2ED
-P 3200 5200
-F 0 "R9" H 3270 5246 50  0000 L CNN
-F 1 "33K" H 3270 5155 50  0000 L CNN
-F 2 "" V 3130 5200 50  0001 C CNN
-F 3 "~" H 3200 5200 50  0001 C CNN
-	1    3200 5200
-	1    0    0    -1
-$EndComp
-$Comp
-L Device:R R10
-U 1 1 605918DA
-P 3700 5200
-F 0 "R10" H 3770 5246 50  0000 L CNN
-F 1 "33K" H 3770 5155 50  0000 L CNN
-F 2 "" V 3630 5200 50  0001 C CNN
-F 3 "~" H 3700 5200 50  0001 C CNN
-	1    3700 5200
-	1    0    0    -1
-$EndComp
-$Comp
-L Device:R R11
-U 1 1 60593E64
-P 4200 5200
-F 0 "R11" H 4270 5246 50  0000 L CNN
-F 1 "33K" H 4270 5155 50  0000 L CNN
-F 2 "" V 4130 5200 50  0001 C CNN
-F 3 "~" H 4200 5200 50  0001 C CNN
-	1    4200 5200
-	1    0    0    -1
-$EndComp
-$Comp
-L Device:R R12
-U 1 1 605963B9
-P 4700 5200
-F 0 "R12" H 4770 5246 50  0000 L CNN
-F 1 "33K" H 4770 5155 50  0000 L CNN
-F 2 "" V 4630 5200 50  0001 C CNN
-F 3 "~" H 4700 5200 50  0001 C CNN
-	1    4700 5200
-	1    0    0    -1
-$EndComp
-$Comp
-L Device:R R13
-U 1 1 60598923
-P 5200 5200
-F 0 "R13" H 5270 5246 50  0000 L CNN
-F 1 "33K" H 5270 5155 50  0000 L CNN
-F 2 "" V 5130 5200 50  0001 C CNN
-F 3 "~" H 5200 5200 50  0001 C CNN
-	1    5200 5200
-	1    0    0    -1
-$EndComp
-$Comp
-L Device:R R14
-U 1 1 6059AEC2
-P 5700 5200
-F 0 "R14" H 5770 5246 50  0000 L CNN
-F 1 "33K" H 5770 5155 50  0000 L CNN
-F 2 "" V 5630 5200 50  0001 C CNN
-F 3 "~" H 5700 5200 50  0001 C CNN
-	1    5700 5200
-	1    0    0    -1
-$EndComp
-$Comp
-L Device:R R15
-U 1 1 6059D49F
-P 6200 5200
-F 0 "R15" H 6270 5246 50  0000 L CNN
-F 1 "33K" H 6270 5155 50  0000 L CNN
-F 2 "" V 6130 5200 50  0001 C CNN
-F 3 "~" H 6200 5200 50  0001 C CNN
-	1    6200 5200
-	1    0    0    -1
-$EndComp
 Wire Wire Line
 	3700 5550 3950 5550
@@
 Wire Wire Line
 	1450 6200 1700 6200
-$Comp
-L power:+5V #PWR0105
-U 1 1 6065B2EA
-P 1550 850
-F 0 "#PWR0105" H 1550 700 50  0001 C CNN
-F 1 "+5V" V 1565 978 50  0000 L CNN
-F 2 "" H 1550 850 50  0001 C CNN
-F 3 "" H 1550 850 50  0001 C CNN
-	1    1550 850
-	0    1    1    0
-$EndComp
-$Comp
-L power:GND #PWR0106
-U 1 1 6065B711
-P 1550 1050
-F 0 "#PWR0106" H 1550 800 50  0001 C CNN
-F 1 "GND" V 1555 922 50  0000 R CNN
-F 2 "" H 1550 1050 50  0001 C CNN
-F 3 "" H 1550 1050 50  0001 C CNN
-	1    1550 1050
-	0    -1   -1   0
-$EndComp
-$Comp
-L power:PWR_FLAG #FLG0101
-U 1 1 6065C0B5
-P 1450 850
-F 0 "#FLG0101" H 1450 925 50  0001 C CNN
-F 1 "PWR_FLAG" H 1450 1023 50  0000 C CNN
-F 2 "" H 1450 850 50  0001 C CNN
-F 3 "~" H 1450 850 50  0001 C CNN
-	1    1450 850
-	1    0    0    -1
-$EndComp
-Connection ~ 1450 850
-Wire Wire Line
-	1450 850  1550 850
-$Comp
-L power:PWR_FLAG #FLG0102
-U 1 1 6065DAFE
-P 1450 1050
-F 0 "#FLG0102" H 1450 1125 50  0001 C CNN
-F 1 "PWR_FLAG" H 1450 1223 50  0000 C CNN
-F 2 "" H 1450 1050 50  0001 C CNN
-F 3 "~" H 1450 1050 50  0001 C CNN
-	1    1450 1050
-	-1   0    0    1
-$EndComp
-Connection ~ 1450 1050
-Wire Wire Line
-	1450 1050 1550 1050
-Wire Wire Line
-	1200 850  1450 850
-Wire Wire Line
-	1200 1050 1450 1050
-$Comp
-L Connector:Barrel_Jack J0
-U 1 1 606418E7
-P 900 950
-F 0 "J0" H 957 1275 50  0000 C CNN
-F 1 "Barrel_Jack" H 957 1184 50  0000 C CNN
-F 2 "" H 950 910 50  0001 C CNN
-F 3 "~" H 950 910 50  0001 C CNN
-	1    900  950
-	1    0    0    -1
-$EndComp
 $Comp
 L Sensor_Optical:TEPT4400 Q0
@@
 NoConn ~ 10050 5550
 NoConn ~ 10150 5550
-$Comp
-L Connector:AVR-ISP-10 J2
-U 1 1 6081F6F5
-P 8000 3350
-F 0 "J2" H 7670 3446 50  0000 R CNN
-F 1 "AVR-ISP-10" H 7670 3355 50  0000 R CNN
-F 2 "" V 7750 3400 50  0001 C CNN
-F 3 " ~" H 6725 2800 50  0001 C CNN
-	1    8000 3350
-	1    0    0    -1
-$EndComp
 NoConn ~ 7900 2850
 $Comp
-L power:GND #PWR?
+L power:GND #PWR0113
 U 1 1 608278F7
 P 7900 3750
-F 0 "#PWR?" H 7900 3500 50  0001 C CNN
+F 0 "#PWR0113" H 7900 3500 50  0001 C CNN
 F 1 "GND" H 7905 3577 50  0000 C CNN
 F 2 "" H 7900 3750 50  0001 C CNN
@@
 Wire Wire Line
 	9000 3150 8400 3150
+$Comp
+L Connector:AVR-ISP-10 J2
+U 1 1 6081F6F5
+P 8000 3350
+F 0 "J2" H 7670 3446 50  0000 R CNN
+F 1 "AVR-ISP-10" H 7670 3355 50  0000 R CNN
+F 2 "" V 7750 3400 50  0001 C CNN
+F 3 " ~" H 6725 2800 50  0001 C CNN
+	1    8000 3350
+	1    0    0    -1
+$EndComp
+$Comp
+L power:+5V #PWR0105
+U 1 1 6065B2EA
+P 8300 5650
+F 0 "#PWR0105" H 8300 5500 50  0001 C CNN
+F 1 "+5V" V 8315 5778 50  0000 L CNN
+F 2 "" H 8300 5650 50  0001 C CNN
+F 3 "" H 8300 5650 50  0001 C CNN
+	1    8300 5650
+	0    1    1    0
+$EndComp
+$Comp
+L power:GND #PWR0106
+U 1 1 6065B711
+P 8300 5850
+F 0 "#PWR0106" H 8300 5600 50  0001 C CNN
+F 1 "GND" V 8305 5722 50  0000 R CNN
+F 2 "" H 8300 5850 50  0001 C CNN
+F 3 "" H 8300 5850 50  0001 C CNN
+	1    8300 5850
+	0    -1   -1   0
+$EndComp
+$Comp
+L power:PWR_FLAG #FLG0101
+U 1 1 6065C0B5
+P 8200 5650
+F 0 "#FLG0101" H 8200 5725 50  0001 C CNN
+F 1 "PWR_FLAG" H 8200 5823 50  0000 C CNN
+F 2 "" H 8200 5650 50  0001 C CNN
+F 3 "~" H 8200 5650 50  0001 C CNN
+	1    8200 5650
+	1    0    0    -1
+$EndComp
+Connection ~ 8200 5650
+Wire Wire Line
+	8200 5650 8300 5650
+$Comp
+L power:PWR_FLAG #FLG0102
+U 1 1 6065DAFE
+P 8200 5850
+F 0 "#FLG0102" H 8200 5925 50  0001 C CNN
+F 1 "PWR_FLAG" H 8200 6023 50  0000 C CNN
+F 2 "" H 8200 5850 50  0001 C CNN
+F 3 "~" H 8200 5850 50  0001 C CNN
+	1    8200 5850
+	-1   0    0    1
+$EndComp
+Connection ~ 8200 5850
+Wire Wire Line
+	8200 5850 8300 5850
+Wire Wire Line
+	7950 5650 8200 5650
+Wire Wire Line
+	7950 5850 8200 5850
+$Comp
+L Connector:Barrel_Jack J0
+U 1 1 606418E7
+P 7650 5750
+F 0 "J0" H 7707 6075 50  0000 C CNN
+F 1 "Barrel_Jack" H 7707 5984 50  0000 C CNN
+F 2 "" H 7700 5710 50  0001 C CNN
+F 3 "~" H 7700 5710 50  0001 C CNN
+	1    7650 5750
+	1    0    0    -1
+$EndComp
+Wire Notes Line
+	1550 5050 6650 5050
+Wire Notes Line
+	6650 5050 6650 5400
+Wire Notes Line
+	6650 5400 1550 5400
+Wire Notes Line
+	1550 5400 1550 5050
+Text Notes 6750 5450 1    50   ~ 0
+Fine-tuned
+$Comp
+L Device:R R6
+U 1 1 60583FB3
+P 1700 5200
+F 0 "R6" H 1770 5246 50  0000 L CNN
+F 1 "68K" H 1770 5155 50  0000 L CNN
+F 2 "" V 1630 5200 50  0001 C CNN
+F 3 "~" H 1700 5200 50  0001 C CNN
+	1    1700 5200
+	1    0    0    -1
+$EndComp
+$Comp
+L Device:R R7
+U 1 1 6058A786
+P 2200 5200
+F 0 "R7" H 2270 5246 50  0000 L CNN
+F 1 "47K" H 2270 5155 50  0000 L CNN
+F 2 "" V 2130 5200 50  0001 C CNN
+F 3 "~" H 2200 5200 50  0001 C CNN
+	1    2200 5200
+	1    0    0    -1
+$EndComp
+$Comp
+L Device:R R8
+U 1 1 6058CD3A
+P 2700 5200
+F 0 "R8" H 2770 5246 50  0000 L CNN
+F 1 "100K" H 2770 5155 50  0000 L CNN
+F 2 "" V 2630 5200 50  0001 C CNN
+F 3 "~" H 2700 5200 50  0001 C CNN
+	1    2700 5200
+	1    0    0    -1
+$EndComp
+$Comp
+L Device:R R9
+U 1 1 6058F2ED
+P 3200 5200
+F 0 "R9" H 3270 5246 50  0000 L CNN
+F 1 "180K" H 3270 5155 50  0000 L CNN
+F 2 "" V 3130 5200 50  0001 C CNN
+F 3 "~" H 3200 5200 50  0001 C CNN
+	1    3200 5200
+	1    0    0    -1
+$EndComp
+$Comp
+L Device:R R10
+U 1 1 605918DA
+P 3700 5200
+F 0 "R10" H 3770 5246 50  0000 L CNN
+F 1 "120K" H 3770 5155 50  0000 L CNN
+F 2 "" V 3630 5200 50  0001 C CNN
+F 3 "~" H 3700 5200 50  0001 C CNN
+	1    3700 5200
+	1    0    0    -1
+$EndComp
+$Comp
+L Device:R R11
+U 1 1 60593E64
+P 4200 5200
+F 0 "R11" H 4270 5246 50  0000 L CNN
+F 1 "120K" H 4270 5155 50  0000 L CNN
+F 2 "" V 4130 5200 50  0001 C CNN
+F 3 "~" H 4200 5200 50  0001 C CNN
+	1    4200 5200
+	1    0    0    -1
+$EndComp
+$Comp
+L Device:R R12
+U 1 1 605963B9
+P 4700 5200
+F 0 "R12" H 4770 5246 50  0000 L CNN
+F 1 "120K" H 4770 5155 50  0000 L CNN
+F 2 "" V 4630 5200 50  0001 C CNN
+F 3 "~" H 4700 5200 50  0001 C CNN
+	1    4700 5200
+	1    0    0    -1
+$EndComp
+$Comp
+L Device:R R13
+U 1 1 60598923
+P 5200 5200
+F 0 "R13" H 5270 5246 50  0000 L CNN
+F 1 "100K" H 5270 5155 50  0000 L CNN
+F 2 "" V 5130 5200 50  0001 C CNN
+F 3 "~" H 5200 5200 50  0001 C CNN
+	1    5200 5200
+	1    0    0    -1
+$EndComp
+$Comp
+L Device:R R14
+U 1 1 6059AEC2
+P 5700 5200
+F 0 "R14" H 5770 5246 50  0000 L CNN
+F 1 "100K" H 5770 5155 50  0000 L CNN
+F 2 "" V 5630 5200 50  0001 C CNN
+F 3 "~" H 5700 5200 50  0001 C CNN
+	1    5700 5200
+	1    0    0    -1
+$EndComp
+$Comp
+L Device:R R15
+U 1 1 6059D49F
+P 6200 5200
+F 0 "R15" H 6270 5246 50  0000 L CNN
+F 1 "68K" H 6270 5155 50  0000 L CNN
+F 2 "" V 6130 5200 50  0001 C CNN
+F 3 "~" H 6200 5200 50  0001 C CNN
+	1    6200 5200
+	1    0    0    -1
+$EndComp
 $EndSCHEMATC

Commit message: Add bypass capacitor
Parts:
- added C0: 100n, symbol Device:C
Connections:
- wire segments 115 -> 118
Changed lines of the file:
@@
 L power:+5V #PWR0109
 U 1 1 607CAF72
-P 9700 3950
-F 0 "#PWR0109" H 9700 3800 50  0001 C CNN
-F 1 "+5V" H 9715 4123 50  0000 C CNN
-F 2 "" H 9700 3950 50  0001 C CNN
-F 3 "" H 9700 3950 50  0001 C CNN
-	1    9700 3950
+P 9700 4400
+F 0 "#PWR0109" H 9700 4250 50  0001 C CNN
+F 1 "+5V" H 9715 4573 50  0000 C CNN
+F 2 "" H 9700 4400 50  0001 C CNN
+F 3 "" H 9700 4400 50  0001 C CNN
+	1    9700 4400
 	-1   0    0    1
 $EndComp
@@
 	1    0    0    -1
 $EndComp
+Wire Wire Line
+	9700 3950 9700 4150
+Wire Wire Line
+	9700 4150 9800 4150
+Connection ~ 9700 4150
+Wire Wire Line
+	9700 4150 9700 4400
+$Comp
+L Device:C C0
+U 1 1 60531D74
+P 9950 4150
+F 0 "C0" V 9698 4150 50  0000 C CNN
+F 1 "100n" V 9789 4150 50  0000 C CNN
+F 2 "" H 9988 4000 50  0001 C CNN
+F 3 "~" H 9950 4150 50  0001 C CNN
+	1    9950 4150
+	0    1    1    0
+$EndComp
+$Comp
+L power:GND #PWR?
+U 1 1 6053249A
+P 10100 4150
+F 0 "#PWR?" H 10100 3900 50  0001 C CNN
+F 1 "GND" V 10105 4022 50  0000 R CNN
+F 2 "" H 10100 4150 50  0001 C CNN
+F 3 "" H 10100 4150 50  0001 C CNN
+	1    10100 4150
+	0    -1   -1   0
+$EndComp
 $EndSCHEMATC
